File: 0006_h_field_probe_15mm.brd (EAGLE design)
At the start: 100 x 20 mm, 10 parts

Commit message: Rev A2 improvements
Parts:
- CONN1: device aaa:SMA-142-0701-801 -> aaa:SMA-EDGE-6.5MM
- moved CONN1 0.30 mm to (38.5, 70.0)
Routing:
- net GND: vias 197 -> 199
Changed lines of the file:
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@@
 </autorouter>
 <elements>
-<element name="CONN1" library="aaa" package="SMA-142-0701-801" value="SMA" x="38.8" y="70" smashed="yes" rot="R90">
-<attribute name="NP" value="" x="261.05" y="89.05" size="1.778" layer="27" rot="R90" display="off"/>
-<attribute name="MFG" value="Cinch Connectivity Solutions Johnson" x="261.05" y="89.05" size="1.778" layer="27" rot="R90" display="off"/>
-<attribute name="VALUE" value="SMA" x="261.05" y="89.05" size="1.778" layer="27" rot="R90" display="off"/>
-<attribute name="DIGIKEY" value="J502-ND" x="261.05" y="89.05" size="1.778" layer="27" rot="R90" display="off"/>
-<attribute name="PN" value="142-0701-801" x="261.05" y="89.05" size="1.778" layer="27" rot="R90" display="off"/>
-<attribute name="NAME" x="43.100003125" y="64.699996875" size="0.4064" layer="25" font="vector" rot="R90"/>
+<element name="CONN1" library="aaa" package="SMA-EDGE-6.5MM" value="SMA" x="38.5" y="70" smashed="yes" rot="R90">
+<attribute name="NP" value="" x="260.75" y="89.05" size="1.778" layer="27" rot="R90" display="off"/>
+<attribute name="MFG" value="Cinch Connectivity Solutions Johnson" x="260.75" y="89.05" size="1.778" layer="27" rot="R90" display="off"/>
+<attribute name="VALUE" value="SMA" x="260.75" y="89.05" size="1.778" layer="27" rot="R90" display="off"/>
+<attribute name="DIGIKEY" value="J502-ND" x="260.75" y="89.05" size="1.778" layer="27" rot="R90" display="off"/>
+<attribute name="PN" value="142-0701-801" x="260.75" y="89.05" size="1.778" layer="27" rot="R90" display="off"/>
+<attribute name="NAME" x="42.800003125" y="64.699996875" size="0.4064" layer="25" font="vector" rot="R90"/>
 </element>
 <element name="U$2" library="aaa" package="FRAME-8.5X11-LANDSCAPE" value="FRAME-8.5X11-LANDSCAPE-LET" x="0" y="0">
@@
 <via x="45.33993125" y="69.36006875" extent="1-16" drill="0.254" diameter="0.4064"/>
 <via x="44.06006875" y="70.63993125" extent="1-16" drill="0.254" diameter="0.4064"/>
-<via x="38.8" y="72.6" extent="1-16" drill="0.254" diameter="0.4064"/>
-<via x="38.8" y="67.4" extent="1-16" drill="0.254" diameter="0.4064"/>
+<via x="38.5" y="72.8" extent="1-16" drill="0.254" diameter="0.4064"/>
+<via x="38.5" y="67.2" extent="1-16" drill="0.254" diameter="0.4064"/>
 <via x="42" y="65.6" extent="1-16" drill="0.254" diameter="0.4064"/>
 <via x="42" y="74.4" extent="1-16" drill="0.254" diameter="0.4064"/>
@@
 <via x="118" y="66.9" extent="1-16" drill="0.254" diameter="0.4069"/>
 <via x="118" y="63.9" extent="1-16" drill="0.254" diameter="0.4069"/>
-<via x="37.2" y="65.6" extent="1-16" drill="0.254" diameter="0.4064"/>
-<via x="40.4" y="65.6" extent="1-16" drill="0.254" diameter="0.4064"/>
-<via x="38.8" y="65.6" extent="1-16" drill="0.254" diameter="0.4064"/>
-<via x="37.2" y="74.4" extent="1-16" drill="0.254" diameter="0.4064"/>
-<via x="38.8" y="74.4" extent="1-16" drill="0.254" diameter="0.4064"/>
-<via x="40.4" y="74.4" extent="1-16" drill="0.254" diameter="0.4064"/>
+<via x="37.2" y="67.2" extent="1-16" drill="0.254" diameter="0.4064"/>
+<via x="41" y="67.2" extent="1-16" drill="0.254" diameter="0.4064"/>
+<via x="38.5" y="65.9" extent="1-16" drill="0.254" diameter="0.4064"/>
+<via x="37.2" y="72.8" extent="1-16" drill="0.254" diameter="0.4064"/>
+<via x="38.5" y="74.1" extent="1-16" drill="0.254" diameter="0.4064"/>
+<via x="41" y="72.8" extent="1-16" drill="0.254" diameter="0.4064"/>
 <wire x1="133.567365625" y1="70.655509375" x2="133.567365625" y2="69.344490625" width="0.254" layer="2" curve="348.6"/>
 <wire x1="44" y1="60.6" x2="126" y2="60.6" width="0.68" layer="2"/>
@@
 <wire x1="40" y1="60.6" x2="36.6" y2="64" width="0.68" layer="3" curve="-90"/>
 <wire x1="40" y1="79.4" x2="36.6" y2="76" width="0.68" layer="3" curve="90"/>
-<wire x1="36.6" y1="76" x2="36.6" y2="74.4" width="0.68" layer="3"/>
-<wire x1="36.6" y1="74.4" x2="36.6" y2="65.6" width="0.68" layer="3"/>
-<wire x1="36.6" y1="65.6" x2="36.6" y2="64" width="0.68" layer="3"/>
-<wire x1="37.2" y1="65.6" x2="36.6" y2="65.6" width="0.68" layer="3"/>
-<wire x1="37.2" y1="74.4" x2="36.6" y2="74.4" width="0.68" layer="3"/>
+<wire x1="36.6" y1="76" x2="36.6" y2="72.8" width="0.68" layer="3"/>
+<wire x1="36.6" y1="72.8" x2="36.6" y2="67.2" width="0.68" layer="3"/>
+<wire x1="36.6" y1="67.2" x2="36.6" y2="64" width="0.68" layer="3"/>
+<wire x1="37.2" y1="67.2" x2="36.6" y2="67.2" width="0.68" layer="3"/>
+<wire x1="37.2" y1="72.8" x2="36.6" y2="72.8" width="0.68" layer="3"/>
+<via x="39.8" y="72.8" extent="1-16" drill="0.254" diameter="0.4064"/>
+<via x="39.8" y="67.2" extent="1-16" drill="0.254" diameter="0.4064"/>
 <wire x1="119.528540625" y1="70.65366875" x2="119.528540625" y2="70.65366875" width="0" layer="19" extent="1-16"/>
 <wire x1="120.4" y1="70" x2="119.528540625" y2="70.65366875" width="0" layer="19" extent="1-1"/>
@@
 <signal name="ANT">
 <contactref element="CONN1" pad="2"/>
-<wire x1="38.8" y1="70" x2="44.7" y2="70" width="0.353" layer="1"/>
+<wire x1="38.5" y1="70" x2="44.7" y2="70" width="0.353" layer="1"/>
 <via x="44.7" y="70" extent="1-16" drill="0.254" diameter="0.568"/>
 <wire x1="44.7" y1="70" x2="119.5" y2="70" width="0.235" layer="2"/>
