File: 0006_h_field_probe_15mm.sch (EAGLE design)
At the start: 10 parts

Commit message: Rev A2 improvements
Parts:
- CONN1: device aaa:COAX-CONNECTOR-EDGE-SMA -> aaa:COAX-CONNECTOR-EDGE-SMA-6.5MM
Changed lines of the file:
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@@
 <parts>
 <part name="U$1" library="aaa" deviceset="GND" device=""/>
-<part name="CONN1" library="aaa" deviceset="COAX-CONNECTOR" device="-EDGE-SMA" value="SMA"/>
+<part name="CONN1" library="aaa" deviceset="COAX-CONNECTOR" device="-EDGE-SMA-6.5MM" value="SMA">
+<attribute name="DIGIKEY" value=""/>
+<attribute name="MFG" value=""/>
+<attribute name="PN" value=""/>
+</part>
 <part name="U$2" library="aaa" deviceset="FRAME-8.5X11-LANDSCAPE" device="-LET">
 <attribute name="DOCNUM" value="0006"/>
